File: PCB/KiCAD/Buttons.kicad_sch (KiCad schematic)
At the start: 12 parts, among them SW1 A, SW10 Dup, SW11 Dright, SW12 Ddown, SW2 B, SW3 X, SW4 Y, SW5 Start, SW6 L, SW7 R, SW8 Z, SW9 Dleft

Commit message: Assembly and fab upload
Upload schematic pdf and bom csv and ibom html docs
Parts:
- SW1, SW10, SW11, SW12, SW2, SW3, SW4, SW5, SW6, SW7, SW9: DNP (none) -> DNP; Package (none) -> Virtual; VARIANT (none) -> NoVar
- SW8: MPN (none) -> 1825027-5; Manufacturer (none) -> TE Connectivity ALCOSWITCH Switches; Package (none) -> Through-hole; VARIANT (none) -> NoVar
Changed lines of the file:
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@@
+      (effects (font (size 1.27 1.27)) hide)
+    )
+    (property "MPN" "" (id 4) (at 203.2 77.47 0)
+      (effects (font (size 1.27 1.27)) hide)
+    )
+    (property "Manufacturer" "" (id 5) (at 203.2 77.47 0)
+      (effects (font (size 1.27 1.27)) hide)
+    )
+    (property "Package" "Virtual" (id 6) (at 203.2 77.47 0)
+      (effects (font (size 1.27 1.27)) hide)
+    )
+    (property "VARIANT" "NoVar" (id 7) (at 203.2 77.47 0)
+      (effects (font (size 1.27 1.27)) hide)
+    )
+    (property "DNP" "DNP" (id 8) (at 203.2 77.47 0)
       (effects (font (size 1.27 1.27)) hide)
     )
@@
       (effects (font (size 1.27 1.27)) hide)
     )
+    (property "MPN" "" (id 4) (at 203.2 107.95 0)
+      (effects (font (size 1.27 1.27)) hide)
+    )
+    (property "Manufacturer" "" (id 5) (at 203.2 107.95 0)
+      (effects (font (size 1.27 1.27)) hide)
+    )
+    (property "Package" "Virtual" (id 6) (at 203.2 107.95 0)
+      (effects (font (size 1.27 1.27)) hide)
+    )
+    (property "VARIANT" "NoVar" (id 7) (at 203.2 107.95 0)
+      (effects (font (size 1.27 1.27)) hide)
+    )
+    (property "DNP" "DNP" (id 8) (at 203.2 107.95 0)
+      (effects (font (size 1.27 1.27)) hide)
+    )
     (pin "1")
     (pin "2")
@@
       (effects (font (size 1.27 1.27)) hide)
     )
+    (property "MPN" "" (id 4) (at 115.57 125.73 0)
+      (effects (font (size 1.27 1.27)) hide)
+    )
+    (property "Manufacturer" "" (id 5) (at 115.57 125.73 0)
+      (effects (font (size 1.27 1.27)) hide)
+    )
+    (property "Package" "Virtual" (id 6) (at 115.57 125.73 0)
+      (effects (font (size 1.27 1.27)) hide)
+    )
+    (property "VARIANT" "NoVar" (id 7) (at 115.57 125.73 0)
+      (effects (font (size 1.27 1.27)) hide)
+    )
+    (property "DNP" "DNP" (id 8) (at 115.57 125.73 0)
+      (effects (font (size 1.27 1.27)) hide)
+    )
     (pin "1")
     (pin "2")
@@
       (effects (font (size 1.27 1.27)) hide)
     )
+    (property "MPN" "" (id 4) (at 203.2 87.63 0)
+      (effects (font (size 1.27 1.27)) hide)
+    )
+    (property "Manufacturer" "" (id 5) (at 203.2 87.63 0)
+      (effects (font (size 1.27 1.27)) hide)
+    )
+    (property "Package" "Virtual" (id 6) (at 203.2 87.63 0)
+      (effects (font (size 1.27 1.27)) hide)
+    )
+    (property "VARIANT" "NoVar" (id 7) (at 203.2 87.63 0)
+      (effects (font (size 1.27 1.27)) hide)
+    )
+    (property "DNP" "DNP" (id 8) (at 203.2 87.63 0)
+      (effects (font (size 1.27 1.27)) hide)
+    )
     (pin "1")
     (pin "2")
@@
       (effects (font (size 1.27 1.27)) hide)
     )
+    (property "MPN" "" (id 4) (at 115.57 137.16 0)
+      (effects (font (size 1.27 1.27)) hide)
+    )
+    (property "Manufacturer" "" (id 5) (at 115.57 137.16 0)
+      (effects (font (size 1.27 1.27)) hide)
+    )
+    (property "Package" "Virtual" (id 6) (at 115.57 137.16 0)
+      (effects (font (size 1.27 1.27)) hide)
+    )
+    (property "VARIANT" "NoVar" (id 7) (at 115.57 137.16 0)
+      (effects (font (size 1.27 1.27)) hide)
+    )
+    (property "DNP" "DNP" (id 8) (at 115.57 137.16 0)
+      (effects (font (size 1.27 1.27)) hide)
+    )
     (pin "1")
     (pin "2")
@@
       (effects (font (size 1.27 1.27)) hide)
     )
+    (property "MPN" "" (id 4) (at 203.2 97.79 0)
+      (effects (font (size 1.27 1.27)) hide)
+    )
+    (property "Manufacturer" "" (id 5) (at 203.2 97.79 0)
+      (effects (font (size 1.27 1.27)) hide)
+    )
+    (property "Package" "Virtual" (id 6) (at 203.2 97.79 0)
+      (effects (font (size 1.27 1.27)) hide)
+    )
+    (property "VARIANT" "NoVar" (id 7) (at 203.2 97.79 0)
+      (effects (font (size 1.27 1.27)) hide)
+    )
+    (property "DNP" "DNP" (id 8) (at 203.2 97.79 0)
+      (effects (font (size 1.27 1.27)) hide)
+    )
     (pin "1")
     (pin "2")
@@
       (effects (font (size 1.27 1.27)) hide)
     )
+    (property "MPN" "" (id 4) (at 203.2 67.31 0)
+      (effects (font (size 1.27 1.27)) hide)
+    )
+    (property "Manufacturer" "" (id 5) (at 203.2 67.31 0)
+      (effects (font (size 1.27 1.27)) hide)
+    )
+    (property "Package" "Virtual" (id 6) (at 203.2 67.31 0)
+      (effects (font (size 1.27 1.27)) hide)
+    )
+    (property "VARIANT" "NoVar" (id 7) (at 203.2 67.31 0)
+      (effects (font (size 1.27 1.27)) hide)
+    )
+    (property "DNP" "DNP" (id 8) (at 203.2 67.31 0)
+      (effects (font (size 1.27 1.27)) hide)
+    )
     (pin "1")
     (pin "2")
@@
       (effects (font (size 1.27 1.27)) hide)
     )
+    (property "MPN" "" (id 4) (at 203.2 55.88 0)
+      (effects (font (size 1.27 1.27)) hide)
+    )
+    (property "Manufacturer" "" (id 5) (at 203.2 55.88 0)
+      (effects (font (size 1.27 1.27)) hide)
+    )
+    (property "Package" "Virtual" (id 6) (at 203.2 55.88 0)
+      (effects (font (size 1.27 1.27)) hide)
+    )
+    (property "VARIANT" "NoVar" (id 7) (at 203.2 55.88 0)
+      (effects (font (size 1.27 1.27)) hide)
+    )
+    (property "DNP" "DNP" (id 8) (at 203.2 55.88 0)
+      (effects (font (size 1.27 1.27)) hide)
+    )
     (pin "1")
     (pin "2")
@@
       (effects (font (size 1.27 1.27)) hide)
     )
+    (property "MPN" "" (id 4) (at 115.57 114.3 0)
+      (effects (font (size 1.27 1.27)) hide)
+    )
+    (property "Manufacturer" "" (id 5) (at 115.57 114.3 0)
+      (effects (font (size 1.27 1.27)) hide)
+    )
+    (property "Package" "Virtual" (id 6) (at 115.57 114.3 0)
+      (effects (font (size 1.27 1.27)) hide)
+    )
+    (property "VARIANT" "NoVar" (id 7) (at 115.57 114.3 0)
+      (effects (font (size 1.27 1.27)) hide)
+    )
+    (property "DNP" "DNP" (id 8) (at 115.57 114.3 0)
+      (effects (font (size 1.27 1.27)) hide)
+    )
     (pin "1")
     (pin "2")
@@
       (effects (font (size 1.27 1.27)) hide)
     )
+    (property "MPN" "" (id 4) (at 203.2 119.38 0)
+      (effects (font (size 1.27 1.27)) hide)
+    )
+    (property "Manufacturer" "" (id 5) (at 203.2 119.38 0)
+      (effects (font (size 1.27 1.27)) hide)
+    )
+    (property "Package" "Virtual" (id 6) (at 203.2 119.38 0)
+      (effects (font (size 1.27 1.27)) hide)
+    )
+    (property "VARIANT" "NoVar" (id 7) (at 203.2 119.38 0)
+      (effects (font (size 1.27 1.27)) hide)
+    )
+    (property "DNP" "DNP" (id 8) (at 203.2 119.38 0)
+      (effects (font (size 1.27 1.27)) hide)
+    )
     (pin "1")
     (pin "2")
@@
       (effects (font (size 1.27 1.27)) (justify left bottom) hide)
     )
+    (property "MPN" "1825027-5" (id 8) (at 182.88 128.27 0)
+      (effects (font (size 1.27 1.27)) hide)
+    )
+    (property "Manufacturer" "TE Connectivity ALCOSWITCH Switches" (id 9) (at 182.88 128.27 0)
+      (effects (font (size 1.27 1.27)) hide)
+    )
+    (property "Package" "Through-hole" (id 10) (at 182.88 128.27 0)
+      (effects (font (size 1.27 1.27)) hide)
+    )
+    (property "VARIANT" "NoVar" (id 11) (at 182.88 128.27 0)
+      (effects (font (size 1.27 1.27)) hide)
+    )
     (pin "1")
     (pin "2")
@@
       (effects (font (size 1.27 1.27)) hide)
     )
+    (property "MPN" "" (id 4) (at 115.57 148.59 0)
+      (effects (font (size 1.27 1.27)) hide)
+    )
+    (property "Manufacturer" "" (id 5) (at 115.57 148.59 0)
+      (effects (font (size 1.27 1.27)) hide)
+    )
+    (property "Package" "Virtual" (id 6) (at 115.57 148.59 0)
+      (effects (font (size 1.27 1.27)) hide)
+    )
+    (property "VARIANT" "NoVar" (id 7) (at 115.57 148.59 0)
+      (effects (font (size 1.27 1.27)) hide)
+    )
+    (property "DNP" "DNP" (id 8) (at 115.57 148.59 0)
+      (effects (font (size 1.27 1.27)) hide)
+    )
