File: PCB/KiCAD/Communications.kicad_sch (KiCad schematic)
At the start: 5 parts, among them Q4 Q_NMOS_GSD

Commit message: Assembly and fab upload
Upload schematic pdf and bom csv and ibom html docs
Parts:
- C2: MPN (none) -> CL10C470JB81PNC; Manufacturer (none) -> Samsung Electro-Mechanics; Package (none) -> 0603; VARIANT (none) -> NoVar
- Q4: LCSC C20917 -> (none); MPN (none) -> T2N7002AK,LM; Manufacturer (none) -> Toshiba Semiconductor and Storage; Package (none) -> SOT-23; VARIANT (none) -> NoVar
- R22: LCSC C22775 -> (none); MPN (none) -> RC0603JR-07750RL; Manufacturer (none) -> YAGEO; Package (none) -> 0603; VARIANT (none) -> NoVar
- R23: LCSC C22775 -> (none); MPN (none) -> RNCP0603FTD1K00; Manufacturer (none) -> Stackpole Electronics Inc; Package (none) -> 0603; VARIANT (none) -> NoVar
- R26: LCSC C22775 -> (none); MPN (none) -> RMCF0603JT220R; Manufacturer (none) -> Stackpole Electronics Inc; Package (none) -> 0603; VARIANT (none) -> NoVar
Changed lines of the file:
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@@
       (effects (font (size 1.27 1.27)) hide)
     )
-    (property "LCSC" "C20917" (id 4) (at 129.54 114.3 0)
+    (property "LCSC" "" (id 4) (at 129.54 114.3 0)
+      (effects (font (size 1.27 1.27)) hide)
+    )
+    (property "MPN" "T2N7002AK,LM" (id 5) (at 129.54 114.3 0)
+      (effects (font (size 1.27 1.27)) hide)
+    )
+    (property "Manufacturer" "Toshiba Semiconductor and Storage" (id 6) (at 129.54 114.3 0)
+      (effects (font (size 1.27 1.27)) hide)
+    )
+    (property "Package" "SOT-23" (id 7) (at 129.54 114.3 0)
+      (effects (font (size 1.27 1.27)) hide)
+    )
+    (property "VARIANT" "NoVar" (id 8) (at 129.54 114.3 0)
       (effects (font (size 1.27 1.27)) hide)
     )
@@
       (effects (font (size 1.27 1.27)) hide)
     )
-    (property "LCSC" "C22775" (id 4) (at 127 82.55 0)
+    (property "LCSC" "" (id 4) (at 127 82.55 0)
       (effects (font (size 1.27 1.27)) hide)
     )
-    (property "MPN" "" (id 5) (at 127 82.55 0)
+    (property "MPN" "RC0603JR-07750RL" (id 5) (at 127 82.55 0)
       (effects (font (size 1.27 1.27)) hide)
     )
-    (property "Manufacturer" "" (id 6) (at 127 82.55 0)
+    (property "Manufacturer" "YAGEO" (id 6) (at 127 82.55 0)
+      (effects (font (size 1.27 1.27)) hide)
+    )
+    (property "Package" "0603" (id 7) (at 127 82.55 0)
+      (effects (font (size 1.27 1.27)) hide)
+    )
+    (property "VARIANT" "NoVar" (id 8) (at 127 82.55 0)
       (effects (font (size 1.27 1.27)) hide)
     )
@@
       (effects (font (size 1.27 1.27)) hide)
     )
-    (property "LCSC" "C22775" (id 4) (at 137.16 88.9 0)
+    (property "LCSC" "" (id 4) (at 137.16 88.9 0)
       (effects (font (size 1.27 1.27)) hide)
     )
-    (property "MPN" "" (id 5) (at 137.16 88.9 0)
+    (property "MPN" "RNCP0603FTD1K00" (id 5) (at 137.16 88.9 0)
       (effects (font (size 1.27 1.27)) hide)
     )
-    (property "Manufacturer" "" (id 6) (at 137.16 88.9 0)
+    (property "Manufacturer" "Stackpole Electronics Inc" (id 6) (at 137.16 88.9 0)
+      (effects (font (size 1.27 1.27)) hide)
+    )
+    (property "Package" "0603" (id 7) (at 137.16 88.9 0)
+      (effects (font (size 1.27 1.27)) hide)
+    )
+    (property "VARIANT" "NoVar" (id 8) (at 137.16 88.9 0)
       (effects (font (size 1.27 1.27)) hide)
     )
@@
     )
     (property "Datasheet" "~" (id 3) (at 144.78 96.52 0)
+      (effects (font (size 1.27 1.27)) hide)
+    )
+    (property "MPN" "CL10C470JB81PNC" (id 4) (at 144.78 96.52 0)
+      (effects (font (size 1.27 1.27)) hide)
+    )
+    (property "Manufacturer" "Samsung Electro-Mechanics" (id 5) (at 144.78 96.52 0)
+      (effects (font (size 1.27 1.27)) hide)
+    )
+    (property "Package" "0603" (id 6) (at 144.78 96.52 0)
+      (effects (font (size 1.27 1.27)) hide)
+    )
+    (property "VARIANT" "NoVar" (id 7) (at 144.78 96.52 0)
       (effects (font (size 1.27 1.27)) hide)
     )
@@
       (effects (font (size 1.27 1.27)) hide)
     )
-    (property "LCSC" "C22775" (id 4) (at 147.32 114.3 0)
+    (property "LCSC" "" (id 4) (at 147.32 114.3 0)
       (effects (font (size 1.27 1.27)) hide)
     )
-    (property "MPN" "" (id 5) (at 147.32 114.3 0)
+    (property "MPN" "RMCF0603JT220R" (id 5) (at 147.32 114.3 0)
       (effects (font (size 1.27 1.27)) hide)
     )
-    (property "Manufacturer" "" (id 6) (at 147.32 114.3 0)
+    (property "Manufacturer" "Stackpole Electronics Inc" (id 6) (at 147.32 114.3 0)
       (effects (font (size 1.27 1.27)) hide)
     )
+    (property "Package" "0603" (id 7) (at 147.32 114.3 0)
+      (effects (font (size 1.27 1.27)) hide)
+    )
+    (property "VARIANT" "NoVar" (id 8) (at 147.32 114.3 0)
+      (effects (font (size 1.27 1.27)) hide)
+    )
