File: PCB/KiCAD/Miscellaneous.kicad_sch (KiCad schematic)
At the start: 9 parts

Commit message: Assembly and fab upload
Upload schematic pdf and bom csv and ibom html docs
Parts:
- H1, H2, H3, H4, H5, H6, H7, H8, H9: DNP (none) -> DNP; Package (none) -> Mechanical; VARIANT (none) -> NoVar
Changed lines of the file:
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@@
+      (effects (font (size 1.27 1.27)) hide)
+    )
+    (property "MPN" "" (id 4) (at 139.7 82.55 0)
+      (effects (font (size 1.27 1.27)) hide)
+    )
+    (property "Manufacturer" "" (id 5) (at 139.7 82.55 0)
+      (effects (font (size 1.27 1.27)) hide)
+    )
+    (property "Package" "Mechanical" (id 6) (at 139.7 82.55 0)
+      (effects (font (size 1.27 1.27)) hide)
+    )
+    (property "VARIANT" "NoVar" (id 7) (at 139.7 82.55 0)
+      (effects (font (size 1.27 1.27)) hide)
+    )
+    (property "DNP" "DNP" (id 8) (at 139.7 82.55 0)
       (effects (font (size 1.27 1.27)) hide)
     )
@@
       (effects (font (size 1.27 1.27)) hide)
     )
+    (property "MPN" "" (id 4) (at 139.7 120.65 0)
+      (effects (font (size 1.27 1.27)) hide)
+    )
+    (property "Manufacturer" "" (id 5) (at 139.7 120.65 0)
+      (effects (font (size 1.27 1.27)) hide)
+    )
+    (property "Package" "Mechanical" (id 6) (at 139.7 120.65 0)
+      (effects (font (size 1.27 1.27)) hide)
+    )
+    (property "VARIANT" "NoVar" (id 7) (at 139.7 120.65 0)
+      (effects (font (size 1.27 1.27)) hide)
+    )
+    (property "DNP" "DNP" (id 8) (at 139.7 120.65 0)
+      (effects (font (size 1.27 1.27)) hide)
+    )
   )
   (symbol (lib_id "Mechanical:MountingHole") (at 139.7 114.3 0) (unit 1)
@@
       (effects (font (size 1.27 1.27)) hide)
     )
+    (property "MPN" "" (id 4) (at 139.7 114.3 0)
+      (effects (font (size 1.27 1.27)) hide)
+    )
+    (property "Manufacturer" "" (id 5) (at 139.7 114.3 0)
+      (effects (font (size 1.27 1.27)) hide)
+    )
+    (property "Package" "Mechanical" (id 6) (at 139.7 114.3 0)
+      (effects (font (size 1.27 1.27)) hide)
+    )
+    (property "VARIANT" "NoVar" (id 7) (at 139.7 114.3 0)
+      (effects (font (size 1.27 1.27)) hide)
+    )
+    (property "DNP" "DNP" (id 8) (at 139.7 114.3 0)
+      (effects (font (size 1.27 1.27)) hide)
+    )
   )
   (symbol (lib_id "Mechanical:MountingHole") (at 139.7 95.25 0) (unit 1)
@@
       (effects (font (size 1.27 1.27)) hide)
     )
+    (property "MPN" "" (id 4) (at 139.7 95.25 0)
+      (effects (font (size 1.27 1.27)) hide)
+    )
+    (property "Manufacturer" "" (id 5) (at 139.7 95.25 0)
+      (effects (font (size 1.27 1.27)) hide)
+    )
+    (property "Package" "Mechanical" (id 6) (at 139.7 95.25 0)
+      (effects (font (size 1.27 1.27)) hide)
+    )
+    (property "VARIANT" "NoVar" (id 7) (at 139.7 95.25 0)
+      (effects (font (size 1.27 1.27)) hide)
+    )
+    (property "DNP" "DNP" (id 8) (at 139.7 95.25 0)
+      (effects (font (size 1.27 1.27)) hide)
+    )
   )
   (symbol (lib_id "Mechanical:MountingHole") (at 139.7 127 0) (unit 1)
@@
       (effects (font (size 1.27 1.27)) hide)
     )
+    (property "MPN" "" (id 4) (at 139.7 127 0)
+      (effects (font (size 1.27 1.27)) hide)
+    )
+    (property "Manufacturer" "" (id 5) (at 139.7 127 0)
+      (effects (font (size 1.27 1.27)) hide)
+    )
+    (property "Package" "Mechanical" (id 6) (at 139.7 127 0)
+      (effects (font (size 1.27 1.27)) hide)
+    )
+    (property "VARIANT" "NoVar" (id 7) (at 139.7 127 0)
+      (effects (font (size 1.27 1.27)) hide)
+    )
+    (property "DNP" "DNP" (id 8) (at 139.7 127 0)
+      (effects (font (size 1.27 1.27)) hide)
+    )
   )
   (symbol (lib_id "Mechanical:MountingHole") (at 139.7 101.6 0) (unit 1)
@@
       (effects (font (size 1.27 1.27)) hide)
     )
+    (property "MPN" "" (id 4) (at 139.7 101.6 0)
+      (effects (font (size 1.27 1.27)) hide)
+    )
+    (property "Manufacturer" "" (id 5) (at 139.7 101.6 0)
+      (effects (font (size 1.27 1.27)) hide)
+    )
+    (property "Package" "Mechanical" (id 6) (at 139.7 101.6 0)
+      (effects (font (size 1.27 1.27)) hide)
+    )
+    (property "VARIANT" "NoVar" (id 7) (at 139.7 101.6 0)
+      (effects (font (size 1.27 1.27)) hide)
+    )
+    (property "DNP" "DNP" (id 8) (at 139.7 101.6 0)
+      (effects (font (size 1.27 1.27)) hide)
+    )
   )
   (symbol (lib_id "Mechanical:MountingHole") (at 139.7 107.95 0) (unit 1)
@@
       (effects (font (size 1.27 1.27)) hide)
     )
+    (property "MPN" "" (id 4) (at 139.7 107.95 0)
+      (effects (font (size 1.27 1.27)) hide)
+    )
+    (property "Manufacturer" "" (id 5) (at 139.7 107.95 0)
+      (effects (font (size 1.27 1.27)) hide)
+    )
+    (property "Package" "Mechanical" (id 6) (at 139.7 107.95 0)
+      (effects (font (size 1.27 1.27)) hide)
+    )
+    (property "VARIANT" "NoVar" (id 7) (at 139.7 107.95 0)
+      (effects (font (size 1.27 1.27)) hide)
+    )
+    (property "DNP" "DNP" (id 8) (at 139.7 107.95 0)
+      (effects (font (size 1.27 1.27)) hide)
+    )
   )
   (symbol (lib_id "Mechanical:MountingHole") (at 139.7 88.9 0) (unit 1)
@@
       (effects (font (size 1.27 1.27)) hide)
     )
+    (property "MPN" "" (id 4) (at 139.7 88.9 0)
+      (effects (font (size 1.27 1.27)) hide)
+    )
+    (property "Manufacturer" "" (id 5) (at 139.7 88.9 0)
+      (effects (font (size 1.27 1.27)) hide)
+    )
+    (property "Package" "Mechanical" (id 6) (at 139.7 88.9 0)
+      (effects (font (size 1.27 1.27)) hide)
+    )
+    (property "VARIANT" "NoVar" (id 7) (at 139.7 88.9 0)
+      (effects (font (size 1.27 1.27)) hide)
+    )
+    (property "DNP" "DNP" (id 8) (at 139.7 88.9 0)
+      (effects (font (size 1.27 1.27)) hide)
+    )
   )
   (symbol (lib_id "Mechanical:MountingHole") (at 139.7 76.2 0) (unit 1)
@@
       (effects (font (size 1.27 1.27)) hide)
     )
+    (property "MPN" "" (id 4) (at 139.7 76.2 0)
+      (effects (font (size 1.27 1.27)) hide)
+    )
+    (property "Manufacturer" "" (id 5) (at 139.7 76.2 0)
+      (effects (font (size 1.27 1.27)) hide)
+    )
+    (property "Package" "Mechanical" (id 6) (at 139.7 76.2 0)
+      (effects (font (size 1.27 1.27)) hide)
+    )
+    (property "VARIANT" "NoVar" (id 7) (at 139.7 76.2 0)
+      (effects (font (size 1.27 1.27)) hide)
+    )
+    (property "DNP" "DNP" (id 8) (at 139.7 76.2 0)
+      (effects (font (size 1.27 1.27)) hide)
+    )
