File: PCB/KiCAD/PowerSupply.kicad_sch (KiCad schematic)
At the start: 4 parts, among them U6 AMS1117-3.3

Commit message: Assembly and fab upload
Upload schematic pdf and bom csv and ibom html docs
Parts:
- C16, C18: MPN (none) -> GRM21BR71A106KA73K; Manufacturer (none) -> Murata Electronics; Package (none) -> 0805; VARIANT (none) -> NoVar
- D1: MPN (none) -> CUS10S30,H3F; Manufacturer (none) -> Toshiba Semiconductor and Storage; Package (none) -> SOD-323; VARIANT (none) -> NoVar
- U6: MPN (none) -> AMS1117-3.3; Manufacturer (none) -> UMW; Package (none) -> SOT-223-3; VARIANT (none) -> NoVar
Changed lines of the file:
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@@
+      (effects (font (size 1.27 1.27)) hide)
+    )
+    (property "MPN" "CUS10S30,H3F" (id 4) (at 142.24 100.33 0)
+      (effects (font (size 1.27 1.27)) hide)
+    )
+    (property "Manufacturer" "Toshiba Semiconductor and Storage" (id 5) (at 142.24 100.33 0)
+      (effects (font (size 1.27 1.27)) hide)
+    )
+    (property "Package" "SOD-323" (id 6) (at 142.24 100.33 0)
+      (effects (font (size 1.27 1.27)) hide)
+    )
+    (property "VARIANT" "NoVar" (id 7) (at 142.24 100.33 0)
       (effects (font (size 1.27 1.27)) hide)
     )
@@
       (effects (font (size 1.27 1.27)) hide)
     )
+    (property "MPN" "AMS1117-3.3" (id 4) (at 125.73 100.33 0)
+      (effects (font (size 1.27 1.27)) hide)
+    )
+    (property "Manufacturer" "UMW" (id 5) (at 125.73 100.33 0)
+      (effects (font (size 1.27 1.27)) hide)
+    )
+    (property "Package" "SOT-223-3" (id 6) (at 125.73 100.33 0)
+      (effects (font (size 1.27 1.27)) hide)
+    )
+    (property "VARIANT" "NoVar" (id 7) (at 125.73 100.33 0)
+      (effects (font (size 1.27 1.27)) hide)
+    )
     (pin "1")
     (pin "2")
@@
     )
     (property "Datasheet" "~" (id 3) (at 152.4 105.41 0)
+      (effects (font (size 1.27 1.27)) hide)
+    )
+    (property "MPN" "GRM21BR71A106KA73K" (id 4) (at 152.4 105.41 0)
+      (effects (font (size 1.27 1.27)) hide)
+    )
+    (property "Manufacturer" "Murata Electronics" (id 5) (at 152.4 105.41 0)
+      (effects (font (size 1.27 1.27)) hide)
+    )
+    (property "Package" "0805" (id 6) (at 152.4 105.41 0)
+      (effects (font (size 1.27 1.27)) hide)
+    )
+    (property "VARIANT" "NoVar" (id 7) (at 152.4 105.41 0)
       (effects (font (size 1.27 1.27)) hide)
     )
@@
       (effects (font (size 1.27 1.27)) hide)
     )
+    (property "MPN" "GRM21BR71A106KA73K" (id 4) (at 107.95 105.41 0)
+      (effects (font (size 1.27 1.27)) hide)
+    )
+    (property "Manufacturer" "Murata Electronics" (id 5) (at 107.95 105.41 0)
+      (effects (font (size 1.27 1.27)) hide)
+    )
+    (property "Package" "0805" (id 6) (at 107.95 105.41 0)
+      (effects (font (size 1.27 1.27)) hide)
+    )
+    (property "VARIANT" "NoVar" (id 7) (at 107.95 105.41 0)
+      (effects (font (size 1.27 1.27)) hide)
+    )
