File: PCB/KiCAD/Rumble.kicad_sch (KiCad schematic)
At the start: 10 parts, among them Q1 Q_NMOS_GSD, Q2 Q_PMOS_GDS, Q3 Q_NMOS_GSD

Commit message: Assembly and fab upload
Upload schematic pdf and bom csv and ibom html docs
Parts:
- D2: MPN (none) -> B5819W; Manufacturer (none) -> Yangzhou Yangjie Electronic Technology Co.,Ltd; Package (none) -> SOD-123; VARIANT (none) -> NoVar
- F1: MPN (none) -> PTS120624V020; Manufacturer (none) -> Eaton - Electronics Division; Package (none) -> 1206; VARIANT (none) -> NoVar
- Q1, Q3: MPN (none) -> AO3400A; Manufacturer (none) -> Alpha & Omega Semiconductor Inc.; Package (none) -> SOT-23; VARIANT (none) -> NoVar
- Q2: MPN (none) -> AO3401A; Manufacturer (none) -> Alpha & Omega Semiconductor Inc.; Package (none) -> SOT-23; VARIANT (none) -> NoVar
- R11, R12: MPN (none) -> RMCF0603FT100R; Manufacturer (none) -> Stackpole Electronics Inc; Package (none) -> 0603; VARIANT (none) -> NoVar
- R13, R14, R15: MPN (none) -> RNCP0603FTD10K0; Manufacturer (none) -> Stackpole Electronics Inc; Package (none) -> 0603; VARIANT (none) -> NoVar
Changed lines of the file:
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@@
       (effects (font (size 1.27 1.27)) hide)
     )
-    (property "MPN" "" (id 5) (at 173.99 119.38 0)
-      (effects (font (size 1.27 1.27)) hide)
-    )
-    (property "Manufacturer" "" (id 6) (at 173.99 119.38 0)
+    (property "MPN" "RNCP0603FTD10K0" (id 5) (at 173.99 119.38 0)
+      (effects (font (size 1.27 1.27)) hide)
+    )
+    (property "Manufacturer" "Stackpole Electronics Inc" (id 6) (at 173.99 119.38 0)
+      (effects (font (size 1.27 1.27)) hide)
+    )
+    (property "Package" "0603" (id 7) (at 173.99 119.38 0)
+      (effects (font (size 1.27 1.27)) hide)
+    )
+    (property "VARIANT" "NoVar" (id 8) (at 173.99 119.38 0)
       (effects (font (size 1.27 1.27)) hide)
     )
@@
       (effects (font (size 1.27 1.27)) hide)
     )
-    (property "MPN" "" (id 5) (at 195.58 95.25 0)
-      (effects (font (size 1.27 1.27)) hide)
-    )
-    (property "Manufacturer" "" (id 6) (at 195.58 95.25 0)
+    (property "MPN" "PTS120624V020" (id 5) (at 195.58 95.25 0)
+      (effects (font (size 1.27 1.27)) hide)
+    )
+    (property "Manufacturer" "Eaton - Electronics Division" (id 6) (at 195.58 95.25 0)
+      (effects (font (size 1.27 1.27)) hide)
+    )
+    (property "Package" "1206" (id 7) (at 195.58 95.25 0)
+      (effects (font (size 1.27 1.27)) hide)
+    )
+    (property "VARIANT" "NoVar" (id 8) (at 195.58 95.25 0)
       (effects (font (size 1.27 1.27)) hide)
     )
@@
     )
     (property "LCSC" "C20917" (id 4) (at 193.04 114.3 0)
+      (effects (font (size 1.27 1.27)) hide)
+    )
+    (property "MPN" "AO3400A" (id 5) (at 193.04 114.3 0)
+      (effects (font (size 1.27 1.27)) hide)
+    )
+    (property "Manufacturer" "Alpha & Omega Semiconductor Inc." (id 6) (at 193.04 114.3 0)
+      (effects (font (size 1.27 1.27)) hide)
+    )
+    (property "Package" "SOT-23" (id 7) (at 193.04 114.3 0)
+      (effects (font (size 1.27 1.27)) hide)
+    )
+    (property "VARIANT" "NoVar" (id 8) (at 193.04 114.3 0)
       (effects (font (size 1.27 1.27)) hide)
     )
@@
       (effects (font (size 1.27 1.27)) hide)
     )
-    (property "MPN" "" (id 5) (at 137.16 93.98 0)
-      (effects (font (size 1.27 1.27)) hide)
-    )
-    (property "Manufacturer" "" (id 6) (at 137.16 93.98 0)
+    (property "MPN" "RNCP0603FTD10K0" (id 5) (at 137.16 93.98 0)
+      (effects (font (size 1.27 1.27)) hide)
+    )
+    (property "Manufacturer" "Stackpole Electronics Inc" (id 6) (at 137.16 93.98 0)
+      (effects (font (size 1.27 1.27)) hide)
+    )
+    (property "Package" "0603" (id 7) (at 137.16 93.98 0)
+      (effects (font (size 1.27 1.27)) hide)
+    )
+    (property "VARIANT" "NoVar" (id 8) (at 137.16 93.98 0)
       (effects (font (size 1.27 1.27)) hide)
     )
@@
       (effects (font (size 1.27 1.27)) hide)
     )
-    (property "MPN" "" (id 5) (at 179.07 114.3 0)
-      (effects (font (size 1.27 1.27)) hide)
-    )
-    (property "Manufacturer" "" (id 6) (at 179.07 114.3 0)
+    (property "MPN" "RMCF0603FT100R" (id 5) (at 179.07 114.3 0)
+      (effects (font (size 1.27 1.27)) hide)
+    )
+    (property "Manufacturer" "Stackpole Electronics Inc" (id 6) (at 179.07 114.3 0)
+      (effects (font (size 1.27 1.27)) hide)
+    )
+    (property "Package" "0603" (id 7) (at 179.07 114.3 0)
+      (effects (font (size 1.27 1.27)) hide)
+    )
+    (property "VARIANT" "NoVar" (id 8) (at 179.07 114.3 0)
       (effects (font (size 1.27 1.27)) hide)
     )
@@
     )
     (property "LCSC" "C20917" (id 4) (at 152.4 88.9 0)
+      (effects (font (size 1.27 1.27)) hide)
+    )
+    (property "MPN" "AO3400A" (id 5) (at 152.4 88.9 0)
+      (effects (font (size 1.27 1.27)) hide)
+    )
+    (property "Manufacturer" "Alpha & Omega Semiconductor Inc." (id 6) (at 152.4 88.9 0)
+      (effects (font (size 1.27 1.27)) hide)
+    )
+    (property "Package" "SOT-23" (id 7) (at 152.4 88.9 0)
+      (effects (font (size 1.27 1.27)) hide)
+    )
+    (property "VARIANT" "NoVar" (id 8) (at 152.4 88.9 0)
       (effects (font (size 1.27 1.27)) hide)
     )
@@
       (effects (font (size 1.27 1.27)) hide)
     )
-    (property "MPN" "" (id 5) (at 142.24 88.9 0)
-      (effects (font (size 1.27 1.27)) hide)
-    )
-    (property "Manufacturer" "" (id 6) (at 142.24 88.9 0)
+    (property "MPN" "RMCF0603FT100R" (id 5) (at 142.24 88.9 0)
+      (effects (font (size 1.27 1.27)) hide)
+    )
+    (property "Manufacturer" "Stackpole Electronics Inc" (id 6) (at 142.24 88.9 0)
+      (effects (font (size 1.27 1.27)) hide)
+    )
+    (property "Package" "0603" (id 7) (at 142.24 88.9 0)
+      (effects (font (size 1.27 1.27)) hide)
+    )
+    (property "VARIANT" "NoVar" (id 8) (at 142.24 88.9 0)
       (effects (font (size 1.27 1.27)) hide)
     )
@@
       (effects (font (size 1.27 1.27)) hide)
     )
-    (property "MPN" "" (id 5) (at 154.94 74.93 0)
-      (effects (font (size 1.27 1.27)) hide)
-    )
-    (property "Manufacturer" "" (id 6) (at 154.94 74.93 0)
+    (property "MPN" "RNCP0603FTD10K0" (id 5) (at 154.94 74.93 0)
+      (effects (font (size 1.27 1.27)) hide)
+    )
+    (property "Manufacturer" "Stackpole Electronics Inc" (id 6) (at 154.94 74.93 0)
+      (effects (font (size 1.27 1.27)) hide)
+    )
+    (property "Package" "0603" (id 7) (at 154.94 74.93 0)
+      (effects (font (size 1.27 1.27)) hide)
+    )
+    (property "VARIANT" "NoVar" (id 8) (at 154.94 74.93 0)
       (effects (font (size 1.27 1.27)) hide)
     )
@@
     )
     (property "LCSC" "C15127" (id 4) (at 165.1 78.74 0)
+      (effects (font (size 1.27 1.27)) hide)
+    )
+    (property "MPN" "AO3401A" (id 5) (at 165.1 78.74 0)
+      (effects (font (size 1.27 1.27)) hide)
+    )
+    (property "Manufacturer" "Alpha & Omega Semiconductor Inc." (id 6) (at 165.1 78.74 0)
+      (effects (font (size 1.27 1.27)) hide)
+    )
+    (property "Package" "SOT-23" (id 7) (at 165.1 78.74 0)
+      (effects (font (size 1.27 1.27)) hide)
+    )
+    (property "VARIANT" "NoVar" (id 8) (at 165.1 78.74 0)
       (effects (font (size 1.27 1.27)) hide)
     )
@@
       (effects (font (size 1.27 1.27)) hide)
     )
-    (property "MPN" "" (id 6) (at 187.96 77.47 0)
-      (effects (font (size 1.27 1.27)) hide)
-    )
-    (property "Manufacturer" "" (id 7) (at 187.96 77.47 0)
-      (effects (font (size 1.27 1.27)) hide)
-    )
+    (property "MPN" "B5819W" (id 6) (at 187.96 77.47 0)
+      (effects (font (size 1.27 1.27)) hide)
+    )
+    (property "Manufacturer" "Yangzhou Yangjie Electronic Technology Co.,Ltd" (id 7) (at 187.96 77.47 0)
+      (effects (font (size 1.27 1.27)) hide)
+    )
+    (property "Package" "SOD-123" (id 8) (at 187.96 77.47 0)
+      (effects (font (size 1.27 1.27)) hide)
+    )
+    (property "VARIANT" "NoVar" (id 9) (at 187.96 77.47 0)
+      (effects (font (size 1.27 1.27)) hide)
+    )
