File: PCB/KiCAD/TriggerPaddles.kicad_sch (KiCad schematic)
At the start: 4 parts, among them SW13 L, SW14 R

Commit message: Assembly and fab upload
Upload schematic pdf and bom csv and ibom html docs
Parts:
- H16, H17: DNP (none) -> DNP; Package (none) -> Mechanical; VARIANT (none) -> NoVar
- SW13, SW14: DNP (none) -> DNP; Package (none) -> Virtual; VARIANT (none) -> NoVar
Changed lines of the file:
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@@
+      (effects (font (size 1.27 1.27)) hide)
+    )
+    (property "MPN" "" (id 4) (at 143.51 93.98 0)
+      (effects (font (size 1.27 1.27)) hide)
+    )
+    (property "Manufacturer" "" (id 5) (at 143.51 93.98 0)
+      (effects (font (size 1.27 1.27)) hide)
+    )
+    (property "Package" "Virtual" (id 6) (at 143.51 93.98 0)
+      (effects (font (size 1.27 1.27)) hide)
+    )
+    (property "VARIANT" "NoVar" (id 7) (at 143.51 93.98 0)
+      (effects (font (size 1.27 1.27)) hide)
+    )
+    (property "DNP" "DNP" (id 8) (at 143.51 93.98 0)
       (effects (font (size 1.27 1.27)) hide)
     )
@@
       (effects (font (size 1.27 1.27)) hide)
     )
+    (property "MPN" "" (id 4) (at 158.75 106.68 0)
+      (effects (font (size 1.27 1.27)) hide)
+    )
+    (property "Manufacturer" "" (id 5) (at 158.75 106.68 0)
+      (effects (font (size 1.27 1.27)) hide)
+    )
+    (property "Package" "Mechanical" (id 6) (at 158.75 106.68 0)
+      (effects (font (size 1.27 1.27)) hide)
+    )
+    (property "VARIANT" "NoVar" (id 7) (at 158.75 106.68 0)
+      (effects (font (size 1.27 1.27)) hide)
+    )
+    (property "DNP" "DNP" (id 8) (at 158.75 106.68 0)
+      (effects (font (size 1.27 1.27)) hide)
+    )
   )
   (symbol (lib_id "Mechanical:MountingHole") (at 158.75 96.52 0) (unit 1)
@@
       (effects (font (size 1.27 1.27)) hide)
     )
+    (property "MPN" "" (id 4) (at 158.75 96.52 0)
+      (effects (font (size 1.27 1.27)) hide)
+    )
+    (property "Manufacturer" "" (id 5) (at 158.75 96.52 0)
+      (effects (font (size 1.27 1.27)) hide)
+    )
+    (property "Package" "Mechanical" (id 6) (at 158.75 96.52 0)
+      (effects (font (size 1.27 1.27)) hide)
+    )
+    (property "VARIANT" "NoVar" (id 7) (at 158.75 96.52 0)
+      (effects (font (size 1.27 1.27)) hide)
+    )
+    (property "DNP" "DNP" (id 8) (at 158.75 96.52 0)
+      (effects (font (size 1.27 1.27)) hide)
+    )
   )
   (symbol (lib_name "SW_Push_2") (lib_id "Switch:SW_Push") (at 143.51 105.41 0) (mirror y) (unit 1)
@@
       (effects (font (size 1.27 1.27)) hide)
     )
+    (property "MPN" "" (id 4) (at 143.51 105.41 0)
+      (effects (font (size 1.27 1.27)) hide)
+    )
+    (property "Manufacturer" "" (id 5) (at 143.51 105.41 0)
+      (effects (font (size 1.27 1.27)) hide)
+    )
+    (property "Package" "Virtual" (id 6) (at 143.51 105.41 0)
+      (effects (font (size 1.27 1.27)) hide)
+    )
+    (property "VARIANT" "NoVar" (id 7) (at 143.51 105.41 0)
+      (effects (font (size 1.27 1.27)) hide)
+    )
+    (property "DNP" "DNP" (id 8) (at 143.51 105.41 0)
+      (effects (font (size 1.27 1.27)) hide)
+    )
