File: PCB/KiCAD/TriggerSliders.kicad_sch (KiCad schematic)
At the start: 4 parts

Commit message: Assembly and fab upload
Upload schematic pdf and bom csv and ibom html docs
Parts:
- C3, C7: MPN (none) -> CL10B473KB8NNNC; Manufacturer (none) -> Samsung Electro-Mechanics; Package (none) -> 0603; VARIANT (none) -> NoVar
- RV1, RV2: MPN (none) -> Trigger-Slider; Manufacturer (none) -> Various; Package (none) -> Through-hole; VARIANT (none) -> NoVar
Changed lines of the file:
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@@
+      (effects (font (size 1.27 1.27)) hide)
+    )
+    (property "MPN" "Trigger-Slider" (id 4) (at 119.38 99.06 0)
+      (effects (font (size 1.27 1.27)) hide)
+    )
+    (property "Manufacturer" "Various" (id 5) (at 119.38 99.06 0)
+      (effects (font (size 1.27 1.27)) hide)
+    )
+    (property "Package" "Through-hole" (id 6) (at 119.38 99.06 0)
+      (effects (font (size 1.27 1.27)) hide)
+    )
+    (property "VARIANT" "NoVar" (id 7) (at 119.38 99.06 0)
       (effects (font (size 1.27 1.27)) hide)
     )
@@
       (effects (font (size 1.27 1.27)) hide)
     )
+    (property "MPN" "Trigger-Slider" (id 4) (at 119.38 63.5 0)
+      (effects (font (size 1.27 1.27)) hide)
+    )
+    (property "Manufacturer" "Various" (id 5) (at 119.38 63.5 0)
+      (effects (font (size 1.27 1.27)) hide)
+    )
+    (property "Package" "Through-hole" (id 6) (at 119.38 63.5 0)
+      (effects (font (size 1.27 1.27)) hide)
+    )
+    (property "VARIANT" "NoVar" (id 7) (at 119.38 63.5 0)
+      (effects (font (size 1.27 1.27)) hide)
+    )
     (pin "1")
     (pin "2")
@@
       (effects (font (size 1.27 1.27)) hide)
     )
-    (property "MPN" "" (id 5) (at 139.7 71.12 0)
+    (property "MPN" "CL10B473KB8NNNC" (id 5) (at 139.7 71.12 0)
       (effects (font (size 1.27 1.27)) hide)
     )
-    (property "Manufacturer" "" (id 6) (at 139.7 71.12 0)
+    (property "Manufacturer" "Samsung Electro-Mechanics" (id 6) (at 139.7 71.12 0)
+      (effects (font (size 1.27 1.27)) hide)
+    )
+    (property "Package" "0603" (id 7) (at 139.7 71.12 0)
+      (effects (font (size 1.27 1.27)) hide)
+    )
+    (property "VARIANT" "NoVar" (id 8) (at 139.7 71.12 0)
       (effects (font (size 1.27 1.27)) hide)
     )
@@
       (effects (font (size 1.27 1.27)) hide)
     )
-    (property "MPN" "" (id 5) (at 139.7 106.68 0)
+    (property "MPN" "CL10B473KB8NNNC" (id 5) (at 139.7 106.68 0)
       (effects (font (size 1.27 1.27)) hide)
     )
-    (property "Manufacturer" "" (id 6) (at 139.7 106.68 0)
+    (property "Manufacturer" "Samsung Electro-Mechanics" (id 6) (at 139.7 106.68 0)
       (effects (font (size 1.27 1.27)) hide)
     )
+    (property "Package" "0603" (id 7) (at 139.7 106.68 0)
+      (effects (font (size 1.27 1.27)) hide)
+    )
+    (property "VARIANT" "NoVar" (id 8) (at 139.7 106.68 0)
+      (effects (font (size 1.27 1.27)) hide)
+    )
