File: PCB/KiCAD/flash.kicad_sch (KiCad schematic)
At the start: 4 parts, among them U7 W25Q128JVS

Commit message: Assembly and fab upload
Upload schematic pdf and bom csv and ibom html docs
Parts:
- C17: MPN (none) -> CL05B104KA5NNNC; Manufacturer (none) -> Samsung Electro-Mechanics; Package (none) -> 0402; VARIANT (none) -> NoVar
- R16: MPN (none) -> RMCF0402FT1K00; Manufacturer (none) -> Stackpole Electronics Inc; Package (none) -> 0402; VARIANT (none) -> NoVar
- S1: LCSC (none) -> C318884; MANUFACTURER XKB Industrial Precision -> (none); MPN (none) -> PTS526 SK15 SMTR2 LFS; Manufacturer (none) -> C&K; Package (none) -> SMD; VARIANT (none) -> NoVar
- U7: MPN (none) -> W25Q128JVSIQ TR; Manufacturer (none) -> Winbond Electronics; Package (none) -> 8-SOIC; VARIANT (none) -> NoVar
Changed lines of the file:
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@@
-      (effects (font (size 1.27 1.27)) (justify left bottom) hide)
-    )
-    (property "MANUFACTURER" "XKB Industrial Precision" (id 5) (at 88.9 101.6 0)
       (effects (font (size 1.27 1.27)) (justify left bottom) hide)
     )
@@
     (property "MAXIMUM_PACKAGE_HEIGHT" "1.5mm" (id 7) (at 88.9 101.6 0)
       (effects (font (size 1.27 1.27)) (justify left bottom) hide)
+    )
+    (property "LCSC" "C318884" (id 8) (at 88.9 101.6 0)
+      (effects (font (size 1.27 1.27)) hide)
+    )
+    (property "MPN" "PTS526 SK15 SMTR2 LFS" (id 9) (at 88.9 101.6 0)
+      (effects (font (size 1.27 1.27)) hide)
+    )
+    (property "Manufacturer" "C&K" (id 10) (at 88.9 101.6 0)
+      (effects (font (size 1.27 1.27)) hide)
+    )
+    (property "Package" "SMD" (id 11) (at 88.9 101.6 0)
+      (effects (font (size 1.27 1.27)) hide)
+    )
+    (property "VARIANT" "NoVar" (id 12) (at 88.9 101.6 0)
+      (effects (font (size 1.27 1.27)) hide)
     )
     (pin "A")
@@
     )
     (property "Datasheet" "http://www.winbond.com/resource-files/w25q128jv_dtr%20revc%2003272018%20plus.pdf" (id 3) (at 151.13 91.44 0)
+      (effects (font (size 1.27 1.27)) hide)
+    )
+    (property "MPN" "W25Q128JVSIQ TR" (id 4) (at 151.13 91.44 0)
+      (effects (font (size 1.27 1.27)) hide)
+    )
+    (property "Manufacturer" "Winbond Electronics" (id 5) (at 151.13 91.44 0)
+      (effects (font (size 1.27 1.27)) hide)
+    )
+    (property "Package" "8-SOIC" (id 6) (at 151.13 91.44 0)
+      (effects (font (size 1.27 1.27)) hide)
+    )
+    (property "VARIANT" "NoVar" (id 7) (at 151.13 91.44 0)
       (effects (font (size 1.27 1.27)) hide)
     )
@@
       (effects (font (size 1.27 1.27)) hide)
     )
+    (property "Package" "0402" (id 4) (at 111.76 101.6 0)
+      (effects (font (size 1.27 1.27)) hide)
+    )
+    (property "MPN" "RMCF0402FT1K00" (id 5) (at 111.76 101.6 0)
+      (effects (font (size 1.27 1.27)) hide)
+    )
+    (property "Manufacturer" "Stackpole Electronics Inc" (id 6) (at 111.76 101.6 0)
+      (effects (font (size 1.27 1.27)) hide)
+    )
+    (property "VARIANT" "NoVar" (id 7) (at 111.76 101.6 0)
+      (effects (font (size 1.27 1.27)) hide)
+    )
     (pin "1")
     (pin "2")
@@
       (effects (font (size 1.27 1.27)) hide)
     )
+    (property "MPN" "CL05B104KA5NNNC" (id 4) (at 157.48 69.85 0)
+      (effects (font (size 1.27 1.27)) hide)
+    )
+    (property "Manufacturer" "Samsung Electro-Mechanics" (id 5) (at 157.48 69.85 0)
+      (effects (font (size 1.27 1.27)) hide)
+    )
+    (property "Package" "0402" (id 6) (at 157.48 69.85 0)
+      (effects (font (size 1.27 1.27)) hide)
+    )
+    (property "VARIANT" "NoVar" (id 7) (at 157.48 69.85 0)
+      (effects (font (size 1.27 1.27)) hide)
+    )
